File: RCR-1-Schematic/RCR-1-Schematic.kicad_sch (KiCad schematic)
At the start: 0 parts

Commit message: pretty much complete
Other:
- added sheet Decatrons (decatrons.kicad_sch)
- added sheet Drivers (drivers.kicad_sch)
- added sheet HighVoltage Supply (high_voltage.kicad_sch)
- added sheet Input (input.kicad_sch)
- added sheet Power Supplies (untitled.kicad_sch)
- added sheet Switches (switches.kicad_sch)
- company: (none) -> Nucleonics Corp of America
- title: (none) -> General Scaler-Ratemeter RCR-1 
